File: Box przedni projekt KiCAD/plytka_pionowa.kicad_sch (KiCad schematic)
At the start: 4 parts, among them J16 hdmi diagnostyka, J17 Złącze TE, J2 piny kątowe, J3 Taśma IDC góra

Commit message: Minor changes
Connections:
- net +24F2: now also J17.16 (Pin_16); no longer J17.8 (Pin_8)
- net +5V: now also J17.8 (Pin_8); no longer J17.16 (Pin_16)
Changed lines of the file:
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@@
     (effects (font (size 1.27 1.27)) (justify left bottom))
   )
-  (label "+24F2" (at 191.77 44.45 180)
+  (label "+24F2" (at 191.77 64.77 180)
     (effects (font (size 1.27 1.27)) (justify right bottom))
   )
@@
     (pin "1")
   )
-  (symbol (lib_id "power:+5V") (at 191.77 64.77 90) (unit 1)
-    (in_bom yes) (on_board yes)
-    (property "Reference" "#PWR0137" (id 0) (at 195.58 64.77 0)
-      (effects (font (size 1.27 1.27)) hide)
-    )
-    (property "Value" "+5V" (id 1) (at 186.69 64.77 90))
-    (property "Footprint" "" (id 2) (at 191.77 64.77 0)
-      (effects (font (size 1.27 1.27)) hide)
-    )
-    (property "Datasheet" "" (id 3) (at 191.77 64.77 0)
-      (effects (font (size 1.27 1.27)) hide)
-    )
+  (symbol (lib_id "power:+5V") (at 191.77 44.45 90) (unit 1)
+    (in_bom yes) (on_board yes)
+    (property "Reference" "#PWR0137" (id 0) (at 195.58 44.45 0)
+      (effects (font (size 1.27 1.27)) hide)
+    )
+    (property "Value" "+5V" (id 1) (at 186.69 44.45 90))
+    (property "Footprint" "" (id 2) (at 191.77 44.45 0)
+      (effects (font (size 1.27 1.27)) hide)
+    )
+    (property "Datasheet" "" (id 3) (at 191.77 44.45 0)
+      (effects (font (size 1.27 1.27)) hide)
+    )
