File: Box przedni projekt KiCAD/PUTM_EV_Front_Box_2022.kicad_pcb (KiCad board)
At the start: 2 copper layers, 209.8 x 117.6 mm, 42 parts, among them J10 Conn_ST_STDC14, J11 Conn_ST_STDC14, J12 Conn_ST_STDC14, J13 Conn_ST_STDC14, J14 Diagnostyka, J15 sockety płytka pozioma, J16 hdmi diagnostyka, J17 Złącze TE, J2 piny kątowe, J3 Taśma IDC góra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

Commit message: preproduction review small bug fixes
Parts:
- moved C3 7.74 mm to (237.0, 55.8)
- moved C7 5.42 mm to (231.3, 71.2), turned to 90 degrees
- moved C8 3.45 mm to (229.8, 71.2), turned to 90 degrees
- moved C6 2.12 mm to (228.1, 71.2), turned to 90 degrees
- moved C1 1.29 mm to (241.5, 55.2)
Routing:
- net +5V: track 164.2 -> 180.3 mm
- net /+24F1: track 73.6 -> 81.1 mm
- net GND: vias 535 -> 502

Commit message: Minor changes
Parts:
- moved L1 3.93 mm to (222.5, 69.0)
- moved C4 1.04 mm to (228.5, 66.7)
Connections:
- J17 pad 16: +5V -> /płytka pionowa/+24F2
- J17 pad 8: /płytka pionowa/+24F2 -> +5V
Routing:
- net +5V: track 180.3 -> 94.1 mm, vias 8 -> 6
- net /+24F1: track 81.1 -> 63.3 mm
- net /płytka pionowa/+24F2: track 34.4 -> 31.0 mm
- net Net-(C4-Pad1): track 2.75 -> 0.71 mm
- net /CLK1: track 92.7 -> 90.7 mm
- net /RST3: track 99.8 -> 101.7 mm
- net GND: track 83.9 -> 82.2 mm, vias 502 -> 477
- net /CLK3: track 98.9 -> 100.2 mm
- net /SWD1: track 89.8 -> 88.7 mm
- net /RST1: track 93.4 -> 92.4 mm
- net /SWD2: track 94.9 -> 94.1 mm
- net /SWD3: track 97.9 -> 98.7 mm
- net /RST5: track 113.2 -> 112.5 mm
- net Net-(C4-Pad2): track 3.16 -> 2.46 mm
- net /CLK5: track 119.3 -> 118.7 mm
- added copper zone on F.Cu, net /+24F1

Commit message: .
Parts:
- removed J10, J11, J12, J13, J8: Conn_ST_STDC14, Connector_PinHeader_2.54mm:PinHeader_2x07_P2.54mm_Vertical
- added APPS: 4, Connector_PinHeader_2.54mm:PinHeader_1x05_P2.54mm_Vertical, F.Cu at (79.0, 147.2)
- added EBS: 2, Connector_PinHeader_2.54mm:PinHeader_1x05_P2.54mm_Vertical, F.Cu at (63.0, 147.2)
- added Karta: 3, Connector_PinHeader_2.54mm:PinHeader_1x05_P2.54mm_Vertical, F.Cu at (71.0, 147.2)
- added Telemetria: 5, Connector_PinHeader_2.54mm:PinHeader_1x05_P2.54mm_Vertical, F.Cu at (87.0, 147.2)
- added Wolne: 1, Connector_PinHeader_2.54mm:PinHeader_1x05_P2.54mm_Vertical, F.Cu at (55.0, 147.2)
Routing:
- net /goldpin-hdmi/SWD3: track 71.9 -> 14.6 mm, vias 0 -> 1
- net /goldpin-hdmi/CLK3: track 61.1 -> 13.6 mm
- net +5V: track 94.1 -> 138.8 mm, vias 6 -> 7
- net /goldpin-hdmi/RST3: track 51.9 -> 17.5 mm
- net /goldpin-hdmi/SWD5: track 25.5 -> 58.5 mm, vias 2 -> 1
- net /goldpin-hdmi/CLK5: track 37.4 -> 67.9 mm, vias 1 -> 0
- net /goldpin-hdmi/CLK1: track 20.3 -> 45.1 mm
- net /goldpin-hdmi/CLK4: track 72.7 -> 49.1 mm
- net /goldpin-hdmi/RST5: track 36.4 -> 53.6 mm, vias 1 -> 0
- net /goldpin-hdmi/RST1: track 13.9 -> 28.9 mm
- net /goldpin-hdmi/SWD4: track 60.4 -> 53.4 mm
- net /goldpin-hdmi/SWD2: track 52.3 -> 45.4 mm
- net /goldpin-hdmi/RST4: track 58.0 -> 52.0 mm, vias 0 -> 1
- net /goldpin-hdmi/RST2: track 45.0 -> 40.4 mm
- net /goldpin-hdmi/SWD1: track 22.1 -> 24.1 mm, vias 2 -> 1
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Other:
- board text added: "5V"
- board text added: "CLK"
- board text added: "GND"
- board text added: "RST"
- board text added: "SWD"
