File: Box przedni projekt KiCAD/goldpin-hdmi.kicad_sch (KiCad schematic)
At the start: 7 parts, among them J10 Conn_ST_STDC14, J11 Conn_ST_STDC14, J12 Conn_ST_STDC14, J13 Conn_ST_STDC14, J7 hdmi wurth, J8 Conn_ST_STDC14, J9 Conn_01x02

Commit message: .
Parts:
- removed J10, J11, J12, J13, J8: Conn_ST_STDC14, Connector_PinHeader_2.54mm:PinHeader_2x07_P2.54mm_Vertical, symbol Connector:Conn_ST_STDC14
- removed J9: Conn_01x02, Connector_PinHeader_2.54mm:PinHeader_1x02_P2.54mm_Vertical, symbol Connector_Generic:Conn_01x02
- added J1: APPS, Connector_PinHeader_2.54mm:PinHeader_1x05_P2.54mm_Vertical, symbol Connector:Conn_01x05_Male
- added J10: Conn_01x02, Connector_PinHeader_2.54mm:PinHeader_1x02_P2.54mm_Vertical, symbol Connector_Generic:Conn_01x02
- added J11: Wolne, Connector_PinHeader_2.54mm:PinHeader_1x05_P2.54mm_Vertical, symbol Connector:Conn_01x05_Male
- added J12: Telemetria, Connector_PinHeader_2.54mm:PinHeader_1x05_P2.54mm_Vertical, symbol Connector:Conn_01x05_Male
- added J8: EBS, Connector_PinHeader_2.54mm:PinHeader_1x05_P2.54mm_Vertical, symbol Connector:Conn_01x05_Male
- added J9: Karta, Connector_PinHeader_2.54mm:PinHeader_1x05_P2.54mm_Vertical, symbol Connector:Conn_01x05_Male
Connections:
- net +5V: now also J1.1 (Pin_1), J11.1 (Pin_1), J12.1 (Pin_1), J8.1 (Pin_1), J9.1 (Pin_1)
- net CAN-H: now also J10.1 (Pin_1)
- net CAN-L: now also J10.2 (Pin_2)
- net CLK1: now also J1.2 (Pin_2)
- net CLK2: now also J9.2 (Pin_2)
- net CLK3: now also J12.2 (Pin_2)
- net CLK4: now also J8.2 (Pin_2)
- net CLK5: now also J11.2 (Pin_2)
- net GND: now also J1.3 (Pin_3), J11.3 (Pin_3), J12.3 (Pin_3), J8.3 (Pin_3), J9.3 (Pin_3)
- net RST1: now also J1.5 (Pin_5)
- net RST2: now also J9.5 (Pin_5)
- net RST3: now also J12.5 (Pin_5)
- net RST4: now also J8.5 (Pin_5)
- net RST5: now also J11.5 (Pin_5)
- net SWD1: now also J1.4 (Pin_4)
- net SWD2: now also J9.4 (Pin_4)
- net SWD3: now also J12.4 (Pin_4)
- net SWD4: now also J8.4 (Pin_4)
- net SWD5: now also J11.4 (Pin_4)
