File: PUTM_EV_FRONT_BOX_2022_Plytka_Pozioma/Box przedni projekt KiCAD/PUTM_EV_Front_Box_2022_Płytka_Pozioma.kicad_pcb (KiCad board)
At the start: 2 copper layers, 127 x 75 mm, 11 parts, among them J14 Diagnostyka, J15 sockety płytka pozioma, J4 Sygnały, J5 Zasilanie+CAN, J6 Taśma IDC dolna

Commit message: Final changes
Parts:
- moved H6 2.80 mm to (81.6, 109.9)
- moved H5 2.20 mm to (81.6, 44.9)
Routing:
- net /Z14: track 73.5 -> 75.2 mm
- net /Z12: track 77.5 -> 78.9 mm
- net /Z10: track 81.8 -> 82.9 mm
- net +5V: track 76.9 -> 77.9 mm
- net GND: vias 146 -> 144
Other:
- board size 127 x 75 mm -> 131 x 75 mm
- copper layers 2 -> 4
