File: PUTM_EV_FRONT_BOX_2022_Plytka_Pionowa/Box przedni projekt KiCAD/PUTM_EV_Front_Box_2022_Płytka_Pionowa.kicad_pcb (KiCad board)
At the start: 4 copper layers, 60 x 75 mm, 24 parts, among them J16 hdmi diagnostyka, J17 Złącze TE, J2 piny kątowe, J3 Taśma IDC góra, U1 LM22679TJ-5.0/NOPB

Commit message: 1.0
Parts:
- moved D3 0.18 mm to (149.8, 67.3)
Routing:
- net GND: vias 331 -> 332
Changed lines of the file:
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@@
     (property "Sheetname" "")
     (attr smd)
-    (fp_text reference "C3" (at -2.2158 0.2106) (layer "F.SilkS")
+    (fp_text reference "C3" (at -2.503881 0.175) (layer "F.SilkS")
       (effects (font (size 1 1) (thickness 0.15)))
     )
@@
     (property "Sheetname" "")
     (attr smd)
-    (fp_text reference "C4" (at -0.075 1.425 180) (layer "F.SilkS")
+    (fp_text reference "C4" (at -1.575 1.803881 180) (layer "F.SilkS")
       (effects (font (size 1 1) (thickness 0.15)))
     )
@@
     (property "Sheetname" "")
     (attr smd)
-    (fp_text reference "C6" (at 2.4005 -0.22) (layer "F.SilkS")
+    (fp_text reference "C6" (at -2.518381 0.7834) (layer "F.SilkS")
       (effects (font (size 1 1) (thickness 0.15)))
     )
@@
     (property "Sheetname" "")
     (attr smd)
-    (fp_text reference "C7" (at 2.4412 0.348) (layer "F.SilkS")
+    (fp_text reference "C7" (at 0.992319 1.593) (layer "F.SilkS")
       (effects (font (size 1 1) (thickness 0.15)))
     )
@@
     (property "Sheetname" "")
     (attr smd)
-    (fp_text reference "C8" (at 2.415 0.07) (layer "F.SilkS")
+    (fp_text reference "C8" (at -2.503881 1.175) (layer "F.SilkS")
       (effects (font (size 1 1) (thickness 0.15)))
     )
@@
   )
   (footprint "Diode_SMD:D_SOD-128" (layer "F.Cu")
-    (at 149.925 67.346119 90)
+    (at 149.75 67.346119 90)
     (descr "D_SOD-128 (CFP5 SlimSMAW), https://assets.nexperia.com/documents/outline-drawing/SOD128.pdf")
     (tags "D_SOD-128")
@@
     (property "Sheetname" "")
     (attr through_hole)
-    (fp_text reference "U1" (at 0 0) (layer "F.SilkS")
+    (fp_text reference "U1" (at 6.395 -4.650719) (layer "F.SilkS")
       (effects (font (size 1 1) (thickness 0.15)))
     )
     (fp_text value "LM22679TJ-5.0/NOPB" (at -13.93 -4.5046) (layer "F.SilkS")
-      (effects (font (size 1 1) (thickness 0.15)))
-    )
-    (fp_text user "*" (at -5.08 8.3439) (layer "F.SilkS")
-      (effects (font (size 1 1) (thickness 0.15)))
-    )
-    (fp_text user "*" (at -5.08 8.3439) (layer "F.SilkS")
       (effects (font (size 1 1) (thickness 0.15)))
     )
     (fp_text user "Copyright 2021 Accelerated Designs. All rights reserved." (at 0 0) (layer "Cmts.User")
       (effects (font (size 0.127 0.127) (thickness 0.002)))
-    )
-    (fp_text user "*" (at -5.08 8.3439) (layer "F.Fab")
-      (effects (font (size 1 1) (thickness 0.15)))
     )
     (fp_text user "*" (at -5.08 8.3439) (layer "F.Fab")
@@
   (via (at 127.425 120.296119) (size 0.8) (drill 0.4) (layers "F.Cu" "B.Cu") (free) (net 1))
   (via (at 169.425 70.506119) (size 0.8) (drill 0.4) (layers "F.Cu" "B.Cu") (free) (net 1))
+  (via (at 158 87) (size 0.8) (drill 0.4) (layers "F.Cu" "B.Cu") (free) (net 1))
   (via (at 128.075 65.746119) (size 0.8) (drill 0.4) (layers "F.Cu" "B.Cu") (free) (net 1))
   (via (at 144.325 97.996119) (size 0.8) (drill 0.4) (layers "F.Cu" "B.Cu") (free) (net 1))
@@
     (polygon
       (pts
-        (xy 150.955 71.096119)
-        (xy 152.775 72.646119)
+        (xy 150.973307 71.074624)
+        (xy 152.793307 72.624624)
         (xy 155.884981 72.69523)
         (xy 155.924992 77.19523)
-        (xy 148.905 77.196119)
-        (xy 148.905 69.446119)
+        (xy 148.5 77.196119)
+        (xy 148.5 69.446119)
         (xy 150.955 69.446119)
       )
@@
         (xy 129.825 81.196119)
         (xy 133.125 80.196119)
-        (xy 136.718271 79.073916)
-        (xy 154.818271 79.073916)
+        (xy 136.718271 79.323916)
+        (xy 154.818271 79.323916)
       )
     )
@@
   )
   (zone (net 1) (net_name "GND") (layer "In1.Cu") (hatch edge 0.508)
-    (connect_pads (clearance 0.508))
+    (connect_pads yes (clearance 0.508))
     (min_thickness 0.254) (filled_areas_thickness no)
     (fill yes (thermal_gap 0.508) (thermal_bridge_width 0.508))

Commit message: 1.1
Parts:
- moved C3 3.63 mm to (165.7, 68.9)
- moved G*** 3.03 mm to (161.0, 94.2)
Routing:
- net /+24F1: track 63.3 -> 65.3 mm
- net GND: vias 332 -> 331
- net +5V: vias 44 -> 43

Commit message: Final changes
Parts:
- moved D2 1.60 mm to (156.1, 94.9)
Routing:
- net GND: track 11.4 -> 15.0 mm, vias 331 -> 332
- net /+24F1: track 65.3 -> 64.4 mm
Changed lines of the file:
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@@
       (disableapertmacros false)
       (usegerberextensions true)
-      (usegerberattributes true)
+      (usegerberattributes false)
       (usegerberadvancedattributes false)
       (creategerberjobfile false)
@@
   )
   (footprint "Diode_SMD:D_SOD-323" (layer "F.Cu")
-    (at 154.45 94.946119 180)
+    (at 156.05 94.9 180)
     (descr "SOD-323")
     (tags "SOD-323")
@@
   (gr_line (start 121.825 134.496119) (end 121.625 59.496119) (layer "Edge.Cuts") (width 0.05))
   (gr_line (start 121.625 59.496119) (end 181.625 59.496119) (layer "Edge.Cuts") (width 0.05))
+  (segment (start 159.35 85.7) (end 159.35 83.95) (width 1) (layer "F.Cu") (net 1))
+  (segment (start 158 87.05) (end 159.35 85.7) (width 1) (layer "F.Cu") (net 1))
   (segment (start 159.355 73.744619) (end 159.355 76.866119) (width 0.8) (layer "F.Cu") (net 1))
   (via (at 123.325 75.496119) (size 0.8) (drill 0.4) (layers "F.Cu" "B.Cu") (free) (net 1))
@@
   (via (at 174.325 70.496119) (size 0.8) (drill 0.4) (layers "F.Cu" "B.Cu") (free) (net 1))
   (via (at 144.325 99.096119) (size 0.8) (drill 0.4) (layers "F.Cu" "B.Cu") (free) (net 1))
+  (via (at 159.35 83.95) (size 0.8) (drill 0.4) (layers "F.Cu" "B.Cu") (net 1))
   (via (at 166.525 79.496119) (size 0.8) (drill 0.4) (layers "F.Cu" "B.Cu") (free) (net 1))
   (via (at 159.825 61.736119) (size 0.8) (drill 0.4) (layers "F.Cu" "B.Cu") (net 1))
@@
   (segment (start 176.95 112.771119) (end 176.135 111.956119) (width 0.25) (layer "F.Cu") (net 62))
   (segment (start 155.706584 128.896119) (end 170.625 128.896119) (width 0.25) (layer "F.Cu") (net 62))
-  (segment (start 161.895 81.857621) (end 162.916013 80.836608) (width 1.5) (layer "F.Cu") (net 64))
-  (segment (start 157.2 90.211119) (end 161.895 85.516119) (width 1.5) (layer "F.Cu") (net 64))
-  (segment (start 155.5 94.946119) (end 156.65 94.946119) (width 0.8) (layer "F.Cu") (net 64))
   (segment (start 156.815 71.686119) (end 156.625 71.496119) (width 0.8) (layer "F.Cu") (net 64))
   (segment (start 165.325 71.496119) (end 165.725 71.896119) (width 1) (layer "F.Cu") (net 64))
-  (segment (start 155.95 99.446119) (end 155.300392 100.095727) (width 1.5) (layer "F.Cu") (net 64))
-  (segment (start 161.895 85.516119) (end 161.895 81.857621) (width 1.5) (layer "F.Cu") (net 64))
-  (segment (start 155.300392 100.095727) (end 155.300392 111.104151) (width 1.5) (layer "F.Cu") (net 64))
-  (segment (start 157.2 93.921119) (end 157.2 90.211119) (width 1.5) (layer "F.Cu") (net 64))
-  (segment (start 156.65 94.946119) (end 157.2 94.396119) (width 0.8) (layer "F.Cu") (net 64))
+  (segment (start 161.895 81.896119) (end 165.725 78.066119) (width 1.5) (layer "F.Cu") (net 64))
   (segment (start 156.625 71.496119) (end 164.825 71.496119) (width 1.2) (layer "F.Cu") (net 64))
+  (segment (start 158.6 96.796119) (end 158.6 94.9) (width 1.5) (layer "F.Cu") (net 64))
+  (segment (start 155.300392 100.095727) (end 158.6 96.796119) (width 1.5) (layer "F.Cu") (net 64))
   (segment (start 165.65 71.171119) (end 165.65 69.65) (width 1) (layer "F.Cu") (net 64))
   (segment (start 152.725 71.496119) (end 152.325 71.096119) (width 1.2) (layer "F.Cu") (net 64))
-  (segment (start 165.725 78.066119) (end 165.725 71.896119) (width 1.5) (layer "F.Cu") (net 64))
-  (segment (start 162.916013 80.836608) (end 162.954511 80.836608) (width 1.5) (layer "F.Cu") (net 64))
   (segment (start 164.825 71.496119) (end 165.325 71.496119) (width 1.2) (layer "F.Cu") (net 64))
-  (segment (start 157.2 94.396119) (end 157.2 93.921119) (width 0.8) (layer "F.Cu") (net 64))
+  (segment (start 161.895 85.516119) (end 161.895 81.896119) (width 1.5) (layer "F.Cu") (net 64))
   (segment (start 165.325 71.496119) (end 165.65 71.171119) (width 1) (layer "F.Cu") (net 64))
-  (segment (start 162.954511 80.836608) (end 165.725 78.066119) (width 1.5) (layer "F.Cu") (net 64))
   (segment (start 152.325 71.096119) (end 152.325 69.771119) (width 1.2) (layer "F.Cu") (net 64))
+  (segment (start 157.1 94.9) (end 158.6 94.9) (width 1) (layer "F.Cu") (net 64))
+  (segment (start 158.6 94.9) (end 158.6 88.811119) (width 1.5) (layer "F.Cu") (net 64))
   (segment (start 156.815 73.744619) (end 156.815 71.686119) (width 0.8) (layer "F.Cu") (net 64))
+  (segment (start 158.6 88.811119) (end 161.895 85.516119) (width 1.5) (layer "F.Cu") (net 64))
   (segment (start 156.625 71.496119) (end 152.725 71.496119) (width 1.2) (layer "F.Cu") (net 64))
-  (segment (start 157.2 98.196119) (end 157.2 93.921119) (width 1.5) (layer "F.Cu") (net 64))
-  (segment (start 155.95 99.446119) (end 157.2 98.196119) (width 1.5) (layer "F.Cu") (net 64))
+  (segment (start 155.300392 111.104151) (end 155.300392 100.095727) (width 1.5) (layer "F.Cu") (net 64))
+  (segment (start 165.725 78.066119) (end 165.725 71.896119) (width 1.5) (layer "F.Cu") (net 64))
   (segment (start 158.085 76.181119) (end 158.1 76.196119) (width 0.8) (layer "F.Cu") (net 65))
   (segment (start 158.085 73.744619) (end 158.085 76.181119) (width 0.8) (layer "F.Cu") (net 65))
@@
       )
     )
+  )
+  (zone (net 0) (net_name "") (layer "F.Cu") (hatch edge 0.508)
+    (connect_pads yes (clearance 0))
+    (min_thickness 0.254)
+    (keepout (tracks not_allowed) (vias not_allowed) (pads not_allowed ) (copperpour not_allowed) (footprints allowed))
+    (fill (thermal_gap 0.508) (thermal_bridge_width 0.508) (smoothing chamfer) (radius 10))
+    (polygon
+      (pts
+        (xy 160.8 85.1)
+        (xy 160.1 85.1)
+        (xy 160.1 82.95)
+        (xy 160.8 82.95)
+      )
+    )

Commit message: Added article
Parts:
- moved G*** 10.4 mm to (161.6, 83.9)
Changed lines of the file:
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@@
+      (rotate (xyz 0 0 0))
+    )
+    (model "${KICAD6_3DMODEL_DIR}/Capacitor_SMD.3dshapes/C_0603_1608Metric.step"
+      (offset (xyz 0 0 0))
+      (scale (xyz 1 1 1))
       (rotate (xyz 0 0 0))
     )
@@
       (rotate (xyz 0 0 0))
     )
+    (model "${KICAD6_3DMODEL_DIR}/Capacitor_SMD.3dshapes/C_0603_1608Metric.step"
+      (offset (xyz 0 0 0))
+      (scale (xyz 1 1 1))
+      (rotate (xyz 0 0 0))
+    )
   )
   (footprint "Capacitor_SMD:C_0603_1608Metric" (layer "F.Cu")
@@
       (rotate (xyz 0 0 0))
     )
+    (model "${KICAD6_3DMODEL_DIR}/Capacitor_SMD.3dshapes/C_0603_1608Metric.step"
+      (offset (xyz 0 0 0))
+      (scale (xyz 1 1 1))
+      (rotate (xyz 0 0 0))
+    )
   )
   (footprint "Capacitor_SMD:C_0603_1608Metric" (layer "F.Cu")
@@
       (rotate (xyz 0 0 0))
     )
+    (model "${KICAD6_3DMODEL_DIR}/Capacitor_SMD.3dshapes/C_0603_1608Metric.step"
+      (offset (xyz 0 0 0))
+      (scale (xyz 1 1 1))
+      (rotate (xyz 0 0 0))
+    )
   )
   (footprint "Capacitor_SMD:C_0603_1608Metric" (layer "F.Cu")
@@
       (rotate (xyz 0 0 0))
     )
+    (model "${KICAD6_3DMODEL_DIR}/Capacitor_SMD.3dshapes/C_0603_1608Metric.step"
+      (offset (xyz 0 0 0))
+      (scale (xyz 1 1 1))
+      (rotate (xyz 0 0 0))
+    )
   )
   (footprint "Capacitor_SMD:C_0603_1608Metric" (layer "F.Cu")
@@
       (net 1 "GND") (pintype "passive"))
     (model "${KISYS3DMOD}/Capacitor_SMD.3dshapes/C_0603_1608Metric.wrl"
+      (offset (xyz 0 0 0))
+      (scale (xyz 1 1 1))
+      (rotate (xyz 0 0 0))
+    )
+    (model "${KICAD6_3DMODEL_DIR}/Capacitor_SMD.3dshapes/C_0603_1608Metric.step"
       (offset (xyz 0 0 0))
       (scale (xyz 1 1 1))
@@
       (rotate (xyz 0 0 0))
     )
+    (model "${KICAD6_3DMODEL_DIR}/Diode_SMD.3dshapes/D_SOD-323.step"
+      (offset (xyz 0 0 0))
+      (scale (xyz 1 1 1))
+      (rotate (xyz 0 0 0))
+    )
   )
   (footprint "Diode_SMD:D_SOD-128" (layer "F.Cu")
@@
       (net 1 "GND") (pinfunction "A") (pintype "passive"))
     (model "${KISYS3DMOD}/Diode_SMD.3dshapes/D_SOD-128.wrl"
+      (offset (xyz 0 0 0))
+      (scale (xyz 1 1 1))
+      (rotate (xyz 0 0 0))
+    )
+    (model "${KICAD6_3DMODEL_DIR}/Diode_SMD.3dshapes/D_SOD-123.step"
       (offset (xyz 0 0 0))
       (scale (xyz 1 1 1))
@@
     (pad "8" smd rect locked (at 0 -0.1524) (size 10.414 10.414) (layers "F.Cu" "F.Paste" "F.Mask")
       (net 1 "GND") (pinfunction "DAP") (pintype "power_in"))
+    (model "${KICAD6_3RD_PARTY}/3d/LM22679TJE-5.0_NOPB.stp"
+      (offset (xyz 0 0 0))
+      (scale (xyz 1 1 1))
+      (rotate (xyz 0 0 -90))
+    )
   )
   (footprint "MountingHole:MountingHole_2.2mm_M2_DIN965_Pad" (layer "F.Cu")
@@
     (pad "55" thru_hole circle (at 7.9248 2.3876 225) (size 1.524 1.524) (drill 0.9) (layers *.Cu *.Mask)
       (net 18 "/płytka pionowa/Z13") (pinfunction "Pin_55") (pintype "passive"))
-    (model "C:/Users/przemson/Desktop/AS216-35PN.STEP" hide
-      (opacity 0.3000)      (offset (xyz 0.3302 1.1684 -18.0086))
+    (model "C:/Users/wasyl/Desktop/PUT Motorsport/Przedni box 05.01.20220/Box przedni/model 3d gniazda autosport 55 PIN.STEP"
+      (offset (xyz 0 0 -1))
       (scale (xyz 1 1 1))
-      (rotate (xyz 0 0 180))
-    )
-    (model "C:/Users/wasyl/Desktop/Przedni box 05.01.2022/Box przedni/model 3d gniazda autosport 55 PIN.STEP"
-      (offset (xyz 0 0 0))
-      (scale (xyz 1 1 1))
-      (rotate (xyz 0 90 0))
+      (rotate (xyz 180 90 180))
     )
   )
   (footprint "User_footprints:PUTM_LOGO_35mm" (layer "B.Cu")
-    (at 161 94.25 90)
+    (at 161.630872 83.918254 90)
     (attr through_hole)
     (fp_text reference "G***" (at 0 0 90) (layer "B.SilkS") hide
@@
     (min_thickness 0.254)
     (keepout (tracks not_allowed) (vias not_allowed) (pads not_allowed ) (copperpour not_allowed) (footprints allowed))
-    (fill (thermal_gap 0.508) (thermal_bridge_width 0.508) (smoothing chamfer) (radius 10))
+    (fill (thermal_gap 0.508) (thermal_bridge_width 0.508))
     (polygon
       (pts
