File: Front Box płytka pionowa/Front Box płytka pionowa.kicad_pcb (KiCad board)
At the start: 4 copper layers, 60 x 75 mm, 24 parts, among them J16 hdmi diagnostyka, J17 Złącze TE, J2 piny kątowe, J3 Taśma IDC góra, U1 LM22679TJ-5.0/NOPB

Commit message: Added missing traces
Connections:
- J16 pad 15: unconnected-(J16-Pad15) -> /płytka pionowa/CAN+
- J16 pad 16: unconnected-(J16-Pad16) -> /płytka pionowa/CAN-
Routing:
- net /płytka pionowa/CAN-: track 76.4 -> 85.6 mm
- net /płytka pionowa/CAN+: track 72.4 -> 80.8 mm
- net +5V: track 16.6 -> 13.0 mm, vias 43 -> 44
- net /płytka pionowa/CLK4: track 16.4 -> 17.0 mm, vias 0 -> 2
