File: Front Box płytka pozioma/Front Box płytka pozioma.kicad_sch (KiCad schematic)
At the start: 9 parts, among them J14 Diagnostyka, J15 sockety płytka pozioma, J4 Sygnały, J5 Zasilanie+CAN, J6 Taśma IDC dolna

Commit message: quick revision
Added LED's to horizontal board, distance between sockets fix, Diagnostic Board 5v line delete and compatibility with HDMI fix
Parts:
- added D1: 5v indicator, LED_SMD:LED_0603_1608Metric_Pad1.05x0.95mm_HandSolder, symbol Device:LED
- added D2: 24v indicator, LED_SMD:LED_0603_1608Metric_Pad1.05x0.95mm_HandSolder, symbol Device:LED
- added R1, R2: 480R, Resistor_SMD:R_0603_1608Metric_Pad0.98x0.95mm_HandSolder, symbol Device:R_Small
- renumbered J4 to J1, J5 to J2, J6 to J3, J14 to J4, J15 to J5
Connections:
- net +24F2: now also D2.2 (A)
- net +5V: now also D1.2 (A)
- net CLK1: now also J4.10 (Pin_10); no longer J4.3 (Pin_3)
- net CLK5: now also J4.3 (Pin_3); no longer J4.10 (Pin_10)
- net GND: now also R1.1, R2.2
- net RST1: now also J4.12 (Pin_12); no longer J4.5 (Pin_5)
- net RST5: now also J4.5 (Pin_5); no longer J4.12 (Pin_12)
- net SWD1: now also J4.8 (Pin_8); no longer J4.1 (Pin_1)
- net SWD5: now also J4.1 (Pin_1); no longer J4.8 (Pin_8)
- new net: D2.1 (K), R2.1
- new net: D1.1 (K), R1.2

Commit message: Changed mounting holes to M3 size because Maciej was crying a lot
Parts:
- H1, H2, H3, H4: footprint MountingHole:MountingHole_2.2mm_M2_DIN965_Pad -> MountingHole:MountingHole_3.2mm_M3_DIN965_Pad
Changed lines of the file:
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@@
       (effects (font (size 1.27 1.27)) (justify left))
     )
-    (property "Footprint" "MountingHole:MountingHole_2.2mm_M2_DIN965_Pad" (id 2) (at 233.68 88.9 0)
+    (property "Footprint" "MountingHole:MountingHole_3.2mm_M3_DIN965_Pad" (id 2) (at 233.68 88.9 0)
       (effects (font (size 1.27 1.27)) hide)
     )
@@
     (property "Reference" "H2" (id 0) (at 233.68 100.33 0))
     (property "Value" "MountingHole_Pad" (id 1) (at 233.68 102.235 0))
-    (property "Footprint" "MountingHole:MountingHole_2.2mm_M2_DIN965_Pad" (id 2) (at 233.68 106.68 0)
+    (property "Footprint" "MountingHole:MountingHole_3.2mm_M3_DIN965_Pad" (id 2) (at 233.68 106.68 0)
       (effects (font (size 1.27 1.27)) hide)
     )
@@
     (property "Reference" "H4" (id 0) (at 252.73 100.33 0))
     (property "Value" "MountingHole_Pad" (id 1) (at 252.73 102.235 0))
-    (property "Footprint" "MountingHole:MountingHole_2.2mm_M2_DIN965_Pad" (id 2) (at 252.73 106.68 0)
+    (property "Footprint" "MountingHole:MountingHole_3.2mm_M3_DIN965_Pad" (id 2) (at 252.73 106.68 0)
       (effects (font (size 1.27 1.27)) hide)
     )
@@
     (property "Reference" "H3" (id 0) (at 252.73 82.55 0))
     (property "Value" "MountingHole_Pad" (id 1) (at 252.73 84.455 0))
-    (property "Footprint" "MountingHole:MountingHole_2.2mm_M2_DIN965_Pad" (id 2) (at 252.73 88.9 0)
+    (property "Footprint" "MountingHole:MountingHole_3.2mm_M3_DIN965_Pad" (id 2) (at 252.73 88.9 0)
       (effects (font (size 1.27 1.27)) hide)
     )
@@
     )
     (path "/03b230d8-cf29-41fe-a22c-db7483944d37"
-      (reference "H1") (unit 1) (value "MountingHole_Pad") (footprint "MountingHole:MountingHole_2.2mm_M2_DIN965_Pad")
+      (reference "H1") (unit 1) (value "MountingHole_Pad") (footprint "MountingHole:MountingHole_3.2mm_M3_DIN965_Pad")
     )
     (path "/1e74d489-87b1-4bf3-a418-5f88597a5fa3"
-      (reference "H2") (unit 1) (value "MountingHole_Pad") (footprint "MountingHole:MountingHole_2.2mm_M2_DIN965_Pad")
+      (reference "H2") (unit 1) (value "MountingHole_Pad") (footprint "MountingHole:MountingHole_3.2mm_M3_DIN965_Pad")
     )
     (path "/a3b83521-1599-4b86-a0dd-3e6c958649d3"
-      (reference "H3") (unit 1) (value "MountingHole_Pad") (footprint "MountingHole:MountingHole_2.2mm_M2_DIN965_Pad")
+      (reference "H3") (unit 1) (value "MountingHole_Pad") (footprint "MountingHole:MountingHole_3.2mm_M3_DIN965_Pad")
     )
     (path "/60eefc2a-ef6f-4357-a44f-d842e480f49d"
-      (reference "H4") (unit 1) (value "MountingHole_Pad") (footprint "MountingHole:MountingHole_2.2mm_M2_DIN965_Pad")
+      (reference "H4") (unit 1) (value "MountingHole_Pad") (footprint "MountingHole:MountingHole_3.2mm_M3_DIN965_Pad")
     )
     (path "/4f2de74c-a0a3-419c-86d3-f1056d120362"
